Commit message: delete unnecessary gazebo worlds and small robot model fixes

File: urdf/robot_model.xacro (robot description, xacro)
@@ -20,5 +20,5 @@
         <box size="0.5 0.25 0.15 "/>
         </geometry>
-        <material name="blue"/>
+        <material name="white"/>
         </visual>
         <xacro:inertial_box mass="2" x="0.5" y="0.25" z="0.15" >
@@ -38,5 +38,5 @@
             <box size=".05 .05 .05"/>
         </geometry>
-        <material name="grey"/>
+        <material name="blue"/>
         </visual>
     </link>
@@ -52,5 +52,5 @@
                 <box size=".05 .05 .05"/>
             </geometry>
-            <material name="red"/>
+            <material name="blue"/>
         </visual>
     </link>
@@ -60,5 +60,4 @@
         <parent link="base_link"/>
     </joint>
-  <!-- Define the IMU SENSOR -->
   <link name="imu_link">
     <inertial>

File: urdf/wheel.xacro (robot description, xacro)
@@ -8,5 +8,5 @@
                     <cylinder length="${l}" radius="${r}"/>
                 </geometry>
-                <material name="red"/>
+                <material name="black"/>
             </visual>
             <xacro:inertial_cylinder mass="5" length="${l}" radius="${r}">

Commit message: replace orb_slam launch with config file and octomap params tuning

File: urdf/robot_model.xacro (robot description, xacro)
@@ -6,10 +6,8 @@
 <xacro:include filename="$(find my_robot_simulation_control)/urdf/inertial.urdf.xacro" />
 <xacro:include filename="$(find my_robot_simulation_control)/urdf/setup.gazebo" />
-<!-- cart_robot -->
 <origin xyz="0.0 0.0 0.0" rpy="0.0 0.0 0.0"/>
-    <link name="base_footprint"/>
-    <joint name="base_joint" type="fixed">
-        <origin rpy="0 0 0" xyz="0 0 0.0102"/>
-        <parent link="base_footprint"/>
+    <link name="dummy_link"/>
+    <joint name="dummy_joint" type="fixed">
+        <parent link="dummy_link"/>
         <child link="base_link"/>
     </joint>

Commit message: replace ros control with skid steer drive plugin

File: urdf/robot_model.xacro (robot description, xacro)
@@ -20,5 +20,5 @@
         <material name="white"/>
         </visual>
-        <xacro:inertial_box mass="5" x="0.5" y="0.25" z="0.15" >
+        <xacro:inertial_box mass="10" x="0.5" y="0.25" z="0.15" >
             <origin xyz="0.0 0.0 0.05" rpy="0.0 0.0 0.0"/>
         </xacro:inertial_box>
@@ -32,5 +32,5 @@
     <link name='camera'>
         <visual name='camera_visual'>
-        <origin xyz="0 0 0.05" rpy=" 0 0 0"/>
+        <origin xyz="0 0 0" rpy=" 0 0 0"/>
         <geometry>
             <box size=".05 .05 .05"/>
@@ -40,5 +40,5 @@
     </link>
     <joint type="fixed" name="camera_joint">
-        <origin xyz="0.10 0 0.15" rpy="0 0 0"/>
+        <origin xyz="0.225 0 0.15" rpy="0 0 0"/>
         <child link="camera"/>
         <parent link="base_link"/>
@@ -46,5 +46,5 @@
     <link name="lidar">
         <visual name='lidar_visual'>
-            <origin xyz="0 0 0.05" rpy=" 0 0 0"/>
+            <origin xyz="0 0 0" rpy=" 0 0 0"/>
             <geometry>
                 <box size=".05 .05 .05"/>
@@ -54,5 +54,5 @@
     </link>
     <joint name="lidar_joint" type="fixed">
-        <origin xyz="0.10 0 0.15" rpy="0 0 1.570796"/>
+        <origin xyz="0.225 0 0.15" rpy="0 0 1.570796"/>
         <child link="lidar"/>
         <parent link="base_link"/>
@@ -81,7 +81,7 @@
     <origin xyz="0.25 0 0.1" rpy="0 0 0" />
   </joint>
-    <xacro:wheel side="up_left" x="0.25" y="0.125" z="0" signY="1" signX="1" r = "0.055" l = "0.044" />
-    <xacro:wheel side="up_right" x="0.25" y="0.125" z="0" signY="-1" signX="1" r = "0.055" l = "0.044" />
-    <xacro:wheel side="down_left" x="0.25" y="0.125" z="0" signY="1" signX="-1" r = "0.055" l = "0.044" />
-    <xacro:wheel side="down_right" x="0.25" y="0.125" z="0" signY="-1" signX="-1" r = "0.055" l = "0.044" />
+    <xacro:wheel side="up_left" x="0.12" y="0.15" z="0"/>
+    <xacro:wheel side="up_right" x="0.12" y="-0.15" z="0"/>
+    <xacro:wheel side="down_left" x="-0.12" y="0.15" z="0"/>
+    <xacro:wheel side="down_right" x="-0.12" y="-0.15" z="0"/>
 </robot>

File: urdf/wheel.xacro (robot description, xacro)
@@ -1,41 +1,41 @@
 <?xml version='1.0'?>
-<robot xmlns:xacro="http://www.ros.org/wiki/xacro" name="cart_robot">
-    <xacro:macro name="wheel" params="side x y z signY signX r l">
-        <link name='wheel_${side}_link'>
-            <visual name='wheel_${side}_visual'>
-            <origin xyz="0 0 ${l/2*signY}" rpy="0 0 0"/>
+<robot name="my_robot" xmlns:xacro="http://www.ros.org/wiki/xacro">
+<xacro:macro name="wheel" params="side x y z">
+    <link name='wheel_${side}'>
+        <visual name='wheel_${side}_visual'>
+            <origin xyz="0 0 0" rpy=" 0 0 0"/>
+            <geometry>
+                <cylinder length="0.044" radius="0.055"/>
+            </geometry>
+            <material name="black"/>
+        </visual>
+        <xacro:inertial_cylinder mass="1" length="0.044" radius="0.055">
+            <origin xyz="0 0 0" rpy="0 0 0"/>
+        </xacro:inertial_cylinder>
+        <collision>
+            <origin xyz="0 0 0" rpy="0 0 0"/>
                 <geometry>
-                    <cylinder length="${l}" radius="${r}"/>
+                    <cylinder radius="0.055" length="0.044"/>
                 </geometry>
-                <material name="black"/>
-            </visual>
-            <xacro:inertial_cylinder mass="10" length="${l}" radius="${r}">
-                <origin xyz="0 0 ${l/2*signY}" rpy="0 0 0"/>
-            </xacro:inertial_cylinder>
-            <collision>
-               <origin xyz="0 0 ${l/2*signY}" rpy="0 0 0"/>
-                <geometry>
-                    <cylinder length="${l}" radius="${r}"/>
-                </geometry>
-            </collision>
-        </link>
-        <joint name="wheel_${side}_joint" type="continuous">
-            <origin xyz="${x*signX} ${y*signY} ${-0.15/2}" rpy="1.57 0 0"/>
-            <axis xyz="0 0 1" />
-            <limit effort="50" velocity="100"/>
-            <joint_properties damping="0.5" friction="0.1"/>
-            <child link="wheel_${side}_link"/>
-            <parent link="base_link"/>
+        </collision>
+    </link>
+    <joint name="wheel_${side}_joint" type="continuous">
+        <origin xyz="${x} ${y} ${z}" rpy="${pi/2} 0 ${pi}"/>
+        <child link="wheel_${side}"/>
+        <axis xyz="0 0 1"/>
+        <parent link="base_link"/>
+        <limit effort="50" velocity="100"/>
+        <joint_properties damping="0" friction="0.01"/>
+    </joint>
+    <transmission name="wheel_${side}_trans">
+        <type>transmission_interface/SimpleTransmission</type>
+        <joint name="wheel_${side}_joint">
+            <hardwareInterface>hardware_interface/EffortJointInterface</hardwareInterface>
         </joint>
-        <transmission name="wheel_${side}_trans">
-            <type>transmission_interface/SimpleTransmission</type>
-            <joint name="wheel_${side}_joint">
-                <hardwareInterface>hardware_interface/EffortJointInterface</hardwareInterface>
-            </joint>
-            <actuator name="wheel_${side}_motor">
-                <hardwareInterface>hardware_interface/EffortJointInterface</hardwareInterface>
-                <mechanicalReduction>1</mechanicalReduction>
-            </actuator>
-        </transmission>
-    </xacro:macro>
+        <actuator name="wheel_${side}_motor">
+            <hardwareInterface>hardware_interface/EffortJointInterface</hardwareInterface>
+            <mechanicalReduction>1</mechanicalReduction>
+        </actuator>
+    </transmission>
+</xacro:macro>
 </robot>

Commit message: robot_localization config fixes

File: urdf/robot_model.xacro (robot description, xacro)
@@ -7,9 +7,4 @@
 <xacro:include filename="$(find cart_robot)/urdf/setup.gazebo" />
 <origin xyz="0.0 0.0 0.0" rpy="0.0 0.0 0.0"/>
-    <link name="dummy_link"/>
-    <joint name="dummy_joint" type="fixed">
-        <parent link="dummy_link"/>
-        <child link="base_link"/>
-    </joint>
     <link name='base_link'>
         <visual name='base_visual'>
